Commit message: Added zk_bm1 driver and control

File: ros2/src/bluhmbot/description/ros2_control/diffbot.ros2_control.xacro (robot description, xacro)
@@ -28,3 +28,57 @@
     </ros2_control>
   </xacro:macro>
+  <xacro:macro name="utility_motors_ros2_control" params="name prefix use_mock_hardware">
+    <ros2_control name="${name}brush" type="system">
+      <xacro:unless value="${use_mock_hardware}">
+        <hardware>
+          <plugin>bluhmbot/UtilityMotorHardware</plugin>
+          <!-- Raspberry Pi PWM sysfs params (adjust to your board setup) -->
+          <param name="pwm_in1">19</param>
+          <param name="pwm_in2">15</param>
+          <param name="frequency">2000</param> <!-- 2 kHz -->
+          <param name="invert_dir">false</param>
+          <!-- Effort mapping + simple sim -->
+          <param name="min_effort">0.0</param>
+          <param name="max_effort">0.5</param>
+        </hardware>
+      </xacro:unless>
+      <xacro:if value="${use_mock_hardware}">
+        <hardware>
+          <plugin>mock_components/GenericSystem</plugin>
+          <param name="calculate_dynamics">true</param>
+        </hardware>
+      </xacro:if>
+      <joint name="${prefix}brush_motor">
+        <command_interface name="effort"/>
+	<state_interface name="effort"/>
+	<state_interface name="position"/>
+      </joint>
+    </ros2_control>
+    <ros2_control name="${name}cutter" type="system">
+      <xacro:unless value="${use_mock_hardware}">
+        <hardware>
+          <plugin>bluhmbot/UtilityMotorHardware</plugin>
+          <!-- Raspberry Pi PWM sysfs params (adjust to your board setup) -->
+          <param name="pwm_in1">18</param>
+          <param name="pwm_in2">14</param>
+          <param name="frequency">2000</param> <!-- 2 kHz -->
+          <param name="invert_dir">false</param>
+          <!-- Effort mapping + simple sim -->
+          <param name="min_effort">0.0</param>
+          <param name="max_effort">100.0</param>
+        </hardware>
+      </xacro:unless>
+      <xacro:if value="${use_mock_hardware}">
+        <hardware>
+          <plugin>mock_components/GenericSystem</plugin>
+          <param name="calculate_dynamics">true</param>
+        </hardware>
+      </xacro:if>
+      <joint name="${prefix}cutter_motor">
+        <command_interface name="effort"/>
+	<state_interface name="effort"/>
+	<state_interface name="position"/>
+      </joint>
+    </ros2_control>
+  </xacro:macro>
 </robot>

Commit message: Added zk_bm1 driver and control

File: ros2/src/bluhmbot/description/ros2_control/diffbot.ros2_control.xacro (robot description, xacro)
@@ -28,3 +28,55 @@
     </ros2_control>
   </xacro:macro>
+  <xacro:macro name="utility_motors_ros2_control" params="name prefix use_mock_hardware">
+    <ros2_control name="${name}brush" type="system">
+      <xacro:unless value="${use_mock_hardware}">
+        <hardware>
+          <plugin>bluhmbot/UtilityMotorHardware</plugin>
+          <!-- Raspberry Pi PWM sysfs params (adjust to your board setup) -->
+          <param name="pwm_in1">19</param>
+          <param name="pwm_in2">15</param>
+          <param name="frequency">2000</param> <!-- 2 kHz -->
+          <param name="invert_dir">false</param>
+          <!-- Effort mapping + simple sim -->
+          <param name="min_effort">0.0</param>
+          <param name="max_effort">0.5</param>
+        </hardware>
+      </xacro:unless>
+      <xacro:if value="${use_mock_hardware}">
+        <hardware>
+          <plugin>mock_components/GenericSystem</plugin>
+          <param name="calculate_dynamics">true</param>
+        </hardware>
+      </xacro:if>
+      <joint name="${prefix}brush_motor">
+        <command_interface name="effort"/>
+        <state_interface name="effort"/>
+      </joint>
+    </ros2_control>
+    <ros2_control name="${name}cutter" type="system">
+      <xacro:unless value="${use_mock_hardware}">
+        <hardware>
+          <plugin>bluhmbot/UtilityMotorHardware</plugin>
+          <!-- Raspberry Pi PWM sysfs params (adjust to your board setup) -->
+          <param name="pwm_in1">18</param>
+          <param name="pwm_in2">14</param>
+          <param name="frequency">2000</param> <!-- 2 kHz -->
+          <param name="invert_dir">false</param>
+          <!-- Effort mapping + simple sim -->
+          <param name="min_effort">0.0</param>
+          <param name="max_effort">100.0</param>
+        </hardware>
+      </xacro:unless>
+      <xacro:if value="${use_mock_hardware}">
+        <hardware>
+          <plugin>mock_components/GenericSystem</plugin>
+          <param name="calculate_dynamics">true</param>
+        </hardware>
+      </xacro:if>
+      <joint name="${prefix}cutter_motor">
+        <command_interface name="effort"/>
+        <state_interface name="effort"/>
+      </joint>
+    </ros2_control>
+  </xacro:macro>
 </robot>
